Commit message: feat: 新增 2D 激光雷达（/scan 360 点 10Hz）
- 新增 lidar_link（圆柱外观 50g）+ lidar_joint（fixed, z=0.15）
- Gazebo ray sensor：360 点 × 360°，10Hz，range 0.1~8.0m
- libgazebo_ros_ray_sensor.so 发布 sensor_msgs/LaserScan 到 /scan
- frame_id=lidar_link，robot_state_publisher 自动发布 TF base_link→lidar_link

已知：50g 车顶质量让静止漂移从 0.17mm/s 升至 5.5mm/s，
ray sensor 插件本身不额外增加漂移。40 秒行驶偏移 0.2m 可接受

File: src/robot_description/urdf/diffbot.urdf.xacro (robot description, xacro)
@@ -202,4 +202,61 @@
     </sensor>
   </gazebo>
+  <!-- ========== 激光雷达 ========== -->
+  <link name="lidar_link">
+    <visual>
+      <geometry>
+        <cylinder radius="0.03" length="0.02"/>
+      </geometry>
+      <material name="lidar_color">
+        <color rgba="0.1 0.1 0.8 1"/>
+      </material>
+    </visual>
+    <collision>
+      <geometry>
+        <cylinder radius="0.03" length="0.02"/>
+      </geometry>
+    </collision>
+    <inertial>
+      <mass value="0.05"/>
+      <inertia ixx="0.00001" ixy="0.0" ixz="0.0"
+               iyy="0.00001" iyz="0.0"
+               izz="0.00001"/>
+    </inertial>
+  </link>
+  <joint name="lidar_joint" type="fixed">
+    <origin xyz="0 0 0.15" rpy="0 0 0"/>
+    <parent link="base_link"/>
+    <child link="lidar_link"/>
+  </joint>
+  <!-- ========== Gazebo 激光雷达插件 ========== -->
+  <gazebo reference="lidar_link">
+    <sensor name="lidar" type="ray">
+      <update_rate>10</update_rate>
+      <always_on>true</always_on>
+      <visualize>true</visualize>
+      <ray>
+        <scan>
+          <horizontal>
+            <samples>360</samples>
+            <resolution>1</resolution>
+            <min_angle>-3.14159</min_angle>
+            <max_angle>3.14159</max_angle>
+          </horizontal>
+        </scan>
+        <range>
+          <min>0.10</min>
+          <max>8.0</max>
+          <resolution>0.01</resolution>
+        </range>
+      </ray>
+      <plugin name="lidar_controller" filename="libgazebo_ros_ray_sensor.so">
+        <ros>
+          <remapping>~/out:=/scan</remapping>
+        </ros>
+        <output_type>sensor_msgs/LaserScan</output_type>
+        <frame_name>lidar_link</frame_name>
+      </plugin>
+    </sensor>
+  </gazebo>
     <!-- ========== 差速驱动插件 ========== -->
   <gazebo>
